File: KiCad/MZ700_EMM.sch (KiCad schematic (older format))
At the start: 43 parts, among them J1 INT VCC, J2 EXT 5V, J3 MZ-80K BUS, U1 74LS04, U10 74LS138, U11 74LS138, U12 HM628512LFP-5, U13 74LS11, U14 74LS245, U15 74LS04, U2 74LS14, U3 74LS245, U4 74LS30, U5 74LS193, U6 74LS193, U7 74LS193, U8 74LS193, U9 74LS193

Commit message: Add files via upload
Parts:
- added D4: 1S4, Diode_THT:D_DO-41_SOD81_P10.16mm_Horizontal, symbol Diode:1N4001
- added R3: 10k, Resistor_THT:R_Axial_DIN0207_L6.3mm_D2.5mm_P7.62mm_Horizontal, symbol Device:R
- added S4: SLIDE_SWITCH_3P, Connector_PinHeader_2.54mm:PinHeader_1x03_P2.54mm_Vertical, symbol Memory_RAM2:SLIDE_SWITCH_3P
Connections:
- wire segments 471 -> 480
- no-connect marks 43 -> 41
Other:
- moved on the sheet: BT1, D1, D2, R2, U13C, U15E, U15F

Commit message: Add files via upload
Parts:
- D1, D2: value 1S4 -> 1N4148
- renumbered D4 to D3
Changed lines of the file:
@@
 AR Path="/692AEAAF/69459EED" Ref="D?"  Part="1"
 F 0 "D2" H 16700 8467 50  0000 C CNN
-F 1 "1S4" H 16700 8376 50  0000 C CNN
+F 1 "1N4148" H 16700 8376 50  0000 C CNN
 F 2 "Diode_THT:D_DO-41_SOD81_P10.16mm_Horizontal" H 16700 8075 50  0001 C CNN
 F 3 "http://www.vishay.com/docs/88503/1n4001.pdf" H 16700 8250 50  0001 C CNN
@@
 AR Path="/692AEAAF/69459EF5" Ref="D?"  Part="1"
 F 0 "D1" H 15700 8517 50  0000 C CNN
-F 1 "1S4" H 15700 8426 50  0000 C CNN
+F 1 "1N4148" H 15700 8426 50  0000 C CNN
 F 2 "Diode_THT:D_DO-41_SOD81_P10.16mm_Horizontal" H 15700 8125 50  0001 C CNN
 F 3 "http://www.vishay.com/docs/88503/1n4001.pdf" H 15700 8300 50  0001 C CNN
@@
 P 17150 6350
 AR Path="/6921BBA5/69E446E7" Ref="D?"  Part="1"
-AR Path="/69E446E7" Ref="D4"  Part="1"
+AR Path="/69E446E7" Ref="D3"  Part="1"
 AR Path="/692AEAAF/69E446E7" Ref="D?"  Part="1"
-F 0 "D4" H 17150 6567 50  0000 C CNN
+F 0 "D3" H 17150 6567 50  0000 C CNN
 F 1 "1S4" H 17150 6476 50  0000 C CNN
 F 2 "Diode_THT:D_DO-41_SOD81_P10.16mm_Horizontal" H 17150 6175 50  0001 C CNN
