File: KiCad/MZ700_EMM.kicad_pcb (KiCad board)
At the start: 2 copper layers, 100 x 100 mm, 47 parts, among them J1 INT VCC, J2 EXT 5V, J3 MZ-80K BUS, U1 74LS04, U10 74LS138, U11 74LS138, U12 HM628512LFP-5, U13 74LS11, U14 74LS245, U15 74LS04, U2 74LS14, U3 74LS245, U4 74LS30, U5 74LS193, U6 74LS193, U7 74LS193, U8 74LS193, U9 74LS193

Commit message: Add files via upload
Parts:
- added D4: 1S4, Diode_THT:D_DO-41_SOD81_P10.16mm_Horizontal, F.Cu at (135.1, 97.9)
- added R3: 10k, Resistor_THT:R_Axial_DIN0207_L6.3mm_D2.5mm_P7.62mm_Horizontal, F.Cu at (140.6, 93.9)
- added S4: SLIDE_SWITCH_3P, Connector_PinHeader_2.54mm:PinHeader_1x03_P2.54mm_Vertical, F.Cu at (185.4, 70.5)
Connections:
- U10 pad 4: Net-(R2-Pad2) -> Net-(U10-Pad4)
- U10 pad 5: Net-(R2-Pad2) -> Net-(U10-Pad4)
- U11 pad 4: Net-(R2-Pad2) -> Net-(U10-Pad4)
- U11 pad 5: Net-(R2-Pad2) -> Net-(U10-Pad4)
- U12 pad 29: /x3_WR -> Net-(R3-Pad2)
- U13 pad 10: GND -> Net-(U10-Pad4)
- U13 pad 11: GND -> Net-(U10-Pad4)
- U13 pad 8: (no net) -> Net-(R2-Pad2)
- U13 pad 9: GND -> Net-(U10-Pad4)
- U15 pad 10: (no net) -> Net-(D4-Pad2)
- U15 pad 11: GND -> Net-(U15-Pad11)
- U15 pad 12: (no net) -> Net-(U15-Pad11)
- U15 pad 13: GND -> /x3_WR
- U4 pad 8: Net-(R2-Pad2) -> Net-(U10-Pad4)
Routing:
- net Net-(U10-Pad4): track 0.00 -> 146.7 mm
- net /x3_WR: track 114.6 -> 220.6 mm
- net Net-(D4-Pad1): track 0.00 -> 65.0 mm
- net /x1_WR: track 182.2 -> 126.3 mm, vias 1 -> 3
- net Net-(R3-Pad2): track 0.00 -> 54.6 mm
- net /x3_RD: track 158.8 -> 122.3 mm
- net Net-(R2-Pad2): track 102.1 -> 69.0 mm
- net Net-(S2-Pad2): track 72.1 -> 102.3 mm, vias 0 -> 2
- net Net-(U5-Pad12): track 63.1 -> 36.6 mm
- net GND: track 569.6 -> 544.9 mm
- net Net-(U1-Pad6): track 97.3 -> 73.3 mm
- net Net-(U3-Pad9): track 98.8 -> 121.5 mm
- net Net-(D4-Pad2): track 0.00 -> 22.2 mm
- net Net-(U12-Pad8): track 76.4 -> 55.2 mm
- net /D6: track 139.9 -> 155.3 mm, vias 2 -> 0
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Other:
- board text added: "EMM for 700(MZ-80K) Rev1.2"
- board text added: "RAM"
- board text added: "ROM"
- board text removed: "EMM for 700(MZ-80K)"

Commit message: Add files via upload
Parts:
- D1, D2: value 1S4 -> 1N4148
- renumbered D4 to D3
Other:
- board text added: "1N4148"

Commit message: Add files via upload
Parts:
- removed D3: 1S4, Diode_THT:D_DO-41_SOD81_P10.16mm_Horizontal
- added Q1: 2N7000, Package_TO_SOT_THT:TO-92, F.Cu at (155.8, 72.0)
- R2: value 10k -> 1k
- moved R2 7.94 mm to (162.9, 91.9), turned to 180 degrees
- moved R3 6.29 mm to (135.8, 97.9), turned to 90 degrees
- moved U15 0.15 mm to (106.6, 94.6)
- moved C17 0.13 mm to (103.5, 89.5)
Connections:
- R2 pad 1: Net-(C12-Pad1) -> Net-(Q1-Pad3)
- R2 pad 2: Net-(R2-Pad2) -> Net-(BT1-Pad1)
- R3 pad 1: Net-(C12-Pad1) -> Net-(R3-Pad1)
- R3 pad 2: Net-(R3-Pad2) -> +5V
- S4 pad 1: Net-(D3-Pad1) -> /x3_WR
- S4 pad 2: Net-(R3-Pad2) -> Net-(R3-Pad1)
- U12 pad 22: Net-(R2-Pad2) -> Net-(Q1-Pad3)
- U12 pad 24: Net-(R2-Pad2) -> Net-(U10-Pad4)
- U12 pad 29: Net-(R3-Pad2) -> Net-(R3-Pad1)
- U13 pad 10: Net-(U10-Pad4) -> GND
- U13 pad 11: Net-(U10-Pad4) -> GND
- U13 pad 8: Net-(R2-Pad2) -> (no net)
- U13 pad 9: Net-(U10-Pad4) -> GND
- U15 pad 10: Net-(D3-Pad2) -> (no net)
- U15 pad 11: Net-(U15-Pad11) -> GND
- U15 pad 12: Net-(U15-Pad11) -> (no net)
- U15 pad 13: /x3_WR -> GND
Routing:
- net /x3_WR: track 220.6 -> 126.4 mm
- net Net-(R2-Pad2): track 69.0 -> 0.00 mm
- net Net-(R3-Pad1): track 0.00 -> 68.1 mm
- net Net-(D3-Pad1): track 65.0 -> 0.00 mm
- net /x1_WR: track 126.3 -> 182.7 mm, vias 3 -> 1
- net Net-(R3-Pad2): track 54.6 -> 0.00 mm
- net Net-(U10-Pad4): track 146.7 -> 94.2 mm
- net /D5: track 120.5 -> 162.5 mm, vias 1 -> 0
- net GND: track 544.9 -> 585.5 mm
- net Net-(Q1-Pad3): track 0.00 -> 32.4 mm
- net Net-(U13-Pad6): track 143.6 -> 112.8 mm, vias 0 -> 1
- net /D6: track 155.3 -> 127.1 mm, vias 0 -> 1
- net +5V: track 372.2 -> 399.5 mm
- net /D1: track 134.8 -> 108.8 mm, vias 0 -> 1
- net Net-(U7-Pad12): track 52.5 -> 78.5 mm, vias 0 -> 1
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Other:
- board text added: "1k"
- board text added: "2N7000"
- board text added: "EMM for 700(MZ-80K) Rev1.5"
- board text removed: "1S4"
- board text removed: "EMM for 700(MZ-80K) Rev1.2"
